File: docs/hardware/hardware.kicad_pcb (KiCad board)
At the start: 2 copper layers, 1.4 x 13 mm, 16 parts, among them J1 BASYS_JA, J2 AudioJack2, J3 GAMEPAD, J6 BASYS_JB, J7 GAMEPAD_1, J8 GAMEPAD_2, SW1 LEFT, SW2 UP, SW3 RIGHT, SW4 PRIMARY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

Commit message: final I/O edits
Parts:
- added R2: R, Resistor_THT:R_Axial_DIN0207_L6.3mm_D2.5mm_P7.62mm_Horizontal, F.Cu at (30.5, 45.7)
- moved J7 5.68 mm to (55.9, 25.4)
- moved J8 2.54 mm to (58.4, 58.4)
Connections:
- A1 pad 15: unconnected-(A1-D0/RX-Pad15) -> GP_P1_DOWN
- A1 pad 16: PPU_HBLANK -> GP_P1_BUT_2
- A1 pad 17: GP_P1_DOWN -> GP_P1_BUT_1
- A1 pad 18: GP_P1_BUT_2 -> GP_P1_LEFT
- A1 pad 19: GP_P1_BUT_1 -> GP_P1_UP
- A1 pad 20: GP_P1_LEFT -> GP_P1_RIGHT
- A1 pad 21: GP_P1_UP -> unused
- A1 pad 22: GP_P1_RIGHT -> PPU_HBLANK
- J1 pad 9: unconnected-(J1-Pin_9-Pad9) -> unused
Routing:
- net unused: track 0.00 -> 45.7 mm, vias 0 -> 1
- net PPU_HBLANK: track 50.8 -> 35.6 mm, vias 3 -> 1
- net SPI_SR: track 26.0 -> 38.7 mm, vias 1 -> 3
- net GND: track 59.5 -> 69.7 mm
- net GP_P1_RIGHT: track 15.2 -> 17.8 mm
- net GP_P1_UP: track 10.2 -> 12.7 mm
- net GP_P1_BUT_2: track 10.2 -> 12.7 mm
- net VCC: track 63.5 -> 61.0 mm
- net GP_P2_UP: track 10.2 -> 12.7 mm
- net GP_P2_RIGHT: track 15.2 -> 17.8 mm
- net GP_P2_LEFT: track 5.08 -> 7.62 mm
- net GP_P2_DOWN: track 15.2 -> 17.8 mm
- net GP_P2_BUT_2: track 10.2 -> 12.7 mm
- net GP_P2_BUT_1: track 5.08 -> 7.62 mm
- net GP_P1_LEFT: track 5.08 -> 7.62 mm
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
Commit message: remove pull down resistor for SPI SR and test new SPI transmit
Parts:
- removed R2: R, Resistor_THT:R_Axial_DIN0207_L6.3mm_D2.5mm_P7.62mm_Horizontal
Routing:
- net SPI_SR: track 38.7 -> 26.0 mm, vias 3 -> 1
- net GND: track 69.7 -> 59.5 mm
Changed lines of the file:
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@@
-    )
-  )
-  (footprint "Resistor_THT:R_Axial_DIN0207_L6.3mm_D2.5mm_P7.62mm_Horizontal" (layer "F.Cu")
-    (at 30.48 45.72)
-    (descr "Resistor, Axial_DIN0207 series, Axial, Horizontal, pin pitch=7.62mm, 0.25W = 1/4W, length*diameter=6.3*2.5mm^2, http://cdn-reichelt.de/documents/datenblatt/B400/1_4W%23YAG.pdf")
-    (tags "Resistor Axial_DIN0207 series Axial Horizontal pin pitch 7.62mm 0.25W = 1/4W length 6.3mm diameter 2.5mm")
-    (property "Sheetfile" "hardware.kicad_sch")
-    (property "Sheetname" "")
-    (property "ki_description" "Resistor")
-    (property "ki_keywords" "R res resistor")
-    (attr through_hole)
-    (fp_text reference "R2" (at 0 -2.37) (layer "F.SilkS") hide
-        (effects (font (size 1 1) (thickness 0.15)))
-    )
-    (fp_text value "R" (at 3.81 2.37) (layer "F.Fab") hide
-        (effects (font (size 1 1) (thickness 0.15)))
-    )
-    (fp_text user "${REFERENCE}" (at 3.81 0) (layer "F.Fab")
-        (effects (font (size 1 1) (thickness 0.15)))
-    )
-    (fp_line (start 0.54 -1.37) (end 7.08 -1.37)
-      (stroke (width 0.12) (type solid)) (layer "F.SilkS"))
-    (fp_line (start 0.54 -1.04) (end 0.54 -1.37)
-      (stroke (width 0.12) (type solid)) (layer "F.SilkS"))
-    (fp_line (start 0.54 1.04) (end 0.54 1.37)
-      (stroke (width 0.12) (type solid)) (layer "F.SilkS"))
-    (fp_line (start 0.54 1.37) (end 7.08 1.37)
-      (stroke (width 0.12) (type solid)) (layer "F.SilkS"))
-    (fp_line (start 7.08 -1.37) (end 7.08 -1.04)
-      (stroke (width 0.12) (type solid)) (layer "F.SilkS"))
-    (fp_line (start 7.08 1.37) (end 7.08 1.04)
-      (stroke (width 0.12) (type solid)) (layer "F.SilkS"))
-    (fp_line (start -1.05 -1.5) (end -1.05 1.5)
-      (stroke (width 0.05) (type solid)) (layer "F.CrtYd"))
-    (fp_line (start -1.05 1.5) (end 8.67 1.5)
-      (stroke (width 0.05) (type solid)) (layer "F.CrtYd"))
-    (fp_line (start 8.67 -1.5) (end -1.05 -1.5)
-      (stroke (width 0.05) (type solid)) (layer "F.CrtYd"))
-    (fp_line (start 8.67 1.5) (end 8.67 -1.5)
-      (stroke (width 0.05) (type solid)) (layer "F.CrtYd"))
-    (fp_line (start 0 0) (end 0.66 0)
-      (stroke (width 0.1) (type solid)) (layer "F.Fab"))
-    (fp_line (start 0.66 -1.25) (end 0.66 1.25)
-      (stroke (width 0.1) (type solid)) (layer "F.Fab"))
-    (fp_line (start 0.66 1.25) (end 6.96 1.25)
-      (stroke (width 0.1) (type solid)) (layer "F.Fab"))
-    (fp_line (start 6.96 -1.25) (end 0.66 -1.25)
-      (stroke (width 0.1) (type solid)) (layer "F.Fab"))
-    (fp_line (start 6.96 1.25) (end 6.96 -1.25)
-      (stroke (width 0.1) (type solid)) (layer "F.Fab"))
-    (fp_line (start 7.62 0) (end 6.96 0)
-      (stroke (width 0.1) (type solid)) (layer "F.Fab"))
-    (pad "1" thru_hole circle (at 0 0) (size 1.6 1.6) (drill 0.8) (layers "*.Cu" "*.Mask")
-      (net 6 "GND") (pintype "passive"))
-    (pad "2" thru_hole oval (at 7.62 0) (size 1.6 1.6) (drill 0.8) (layers "*.Cu" "*.Mask")
-      (net 10 "SPI_SR") (pintype "passive"))
-    (model "${KICAD6_3DMODEL_DIR}/Resistor_THT.3dshapes/R_Axial_DIN0207_L6.3mm_D2.5mm_P7.62mm_Horizontal.wrl"
-      (offset (xyz 0 0 0))
-      (scale (xyz 1 1 1))
-      (rotate (xyz 0 0 0))
     )
   )
@@
   (via (at 35.56 63.5) (size 0.8) (drill 0.4) (layers "F.Cu" "B.Cu") (net 4))
   (segment (start 35.56 66.04) (end 35.56 63.5) (width 0.25) (layer "B.Cu") (net 4))
-  (segment (start 27.94 45.72) (end 27.94 38.1) (width 0.25) (layer "F.Cu") (net 6))
   (segment (start 111.76 83.82) (end 109.22 86.36) (width 0.25) (layer "F.Cu") (net 6))
   (segment (start 27.94 20.32) (end 27.94 35.56) (width 0.25) (layer "F.Cu") (net 6))
@@
   (segment (start 27.94 35.56) (end 27.94 38.1) (width 0.25) (layer "F.Cu") (net 6))
   (segment (start 104.26 78.74) (end 106.68 78.74) (width 0.25) (layer "F.Cu") (net 6))
-  (segment (start 30.48 45.72) (end 27.94 45.72) (width 0.25) (layer "F.Cu") (net 6))
   (segment (start 99.06 86.36) (end 99.06 88.9) (width 0.25) (layer "F.Cu") (net 6))
   (segment (start 99.06 88.9) (end 86.36 88.9) (width 0.25) (layer "F.Cu") (net 6))
@@
   (segment (start 45.72 17.78) (end 45.72 20.32) (width 0.25) (layer "B.Cu") (net 9))
   (segment (start 43.18 38.1) (end 38.1 38.1) (width 0.25) (layer "F.Cu") (net 10))
-  (segment (start 38.1 45.72) (end 43.18 45.72) (width 0.25) (layer "F.Cu") (net 10))
   (segment (start 43.18 20.32) (end 43.18 38.1) (width 0.25) (layer "F.Cu") (net 10))
-  (via (at 43.18 38.1) (size 0.8) (drill 0.4) (layers "F.Cu" "B.Cu") (net 10))
   (via (at 43.18 20.32) (size 0.8) (drill 0.4) (layers "F.Cu" "B.Cu") (net 10))
-  (via (at 43.18 45.72) (size 0.8) (drill 0.4) (layers "F.Cu" "B.Cu") (net 10))
-  (segment (start 43.18 45.72) (end 43.18 38.1) (width 0.25) (layer "B.Cu") (net 10))
   (segment (start 43.18 19.3) (end 43.18 20.32) (width 0.25) (layer "B.Cu") (net 10))
   (segment (start 41.66 17.78) (end 43.18 19.3) (width 0.25) (layer "B.Cu") (net 10))
